File: mcu.brd (EAGLE design)
At the start: 100 x 80 mm, 50 parts, among them Q3 DMG3415U-7, SW1 KMR2, SW2 KMR2, U1 MDBT42, U2 AP2112(3.3V), U3 MCP73831T-2ACI/OT, U4 CP2104, U5 MDBT42, X1 4u20317, X2 JSTPH, X3 4u20329, X4 32.768

Commit message: ADD: component and library
Parts:
- removed C10, C11: 0.1uF, microbuilder:0603-NO
- removed C12: 1nF, microbuilder:0603-NO
- removed C13, C9: 300pF, microbuilder:_0603MP
- removed C6, C8: 10µF, microbuilder:0805-NO
- removed C7: 10uf, microbuilder:0805-NO
- removed CHG: ORANGE, microbuilder:CHIPLED_0805_NOOUTLINE
- removed D2: BLUE, microbuilder:CHIPLED_0805_NOOUTLINE
- removed D4: 1N4148, microbuilder:SOD-323
- removed D5: MBR120, microbuilder:SOD-123
- removed FID1, FID3: FIDUCIAL_1MM, microbuilder:FIDUCIAL_1MM
- removed JP1, JP2: (no value), microbuilder:1X01_2MM
- removed L2: 10uH, microbuilder:0805-NO
- removed MS1: FEATHERWING_NODIM, microbuilder:FEATHERWING_NODIM
- removed Q3: DMG3415U-7, microbuilder:SOT23-R
- removed R12: 100k, microbuilder:0603-NO
- removed R6: 2M, microbuilder:0603-NO
- removed R7, R8: 10K, microbuilder:0603-NO
- removed R9: 1K, microbuilder:0603-NO
- removed SJ2: BAT, microbuilder:SOLDERJUMPER_CLOSEDWIRE
- removed SW1, SW2: KMR2, microbuilder:BTN_KMR2_4.6X2.8
- removed TP2: FRST, microbuilder:PAD-1.5X2.0
- removed TP3, TP4: (no value), microbuilder:TESTPOINT_ROUND_2MM
- removed U1, U5: MDBT42, microbuilder:BLE_MODULE_RAYTAC_MDBT42
- removed U2: AP2112(3.3V), microbuilder:SOT23-5
- removed U3: MCP73831T-2ACI/OT, microbuilder:SOT23-5
- removed X1: 4u20317, microbuilder:2X05_1.27MM_BOX_POSTS
- removed X2: JSTPH, microbuilder:JSTPH2
- removed X3: 4u20329, microbuilder:4UCONN_20329_V2
- removed X4: 32.768, adafruit2:XTAL3215
- added C33, C34, C43, C44: 12pF, Nordic_nRF:RESC0402_N
- added C35: 0.8pF, Nordic_nRF:RESC0402_N
- added C36, C37, C40: 100nF, Nordic_nRF:RESC0402_N
- added C38: N.M., Nordic_nRF:RESC0402_N
- added C39: 100pF, Nordic_nRF:RESC0402_N
- added C41: 4.7µF, Nordic_nRF:RESC0603_N
- added C42: 1.0µF, Nordic_nRF:RESC0603_N
- added IC1: MCP73831/OT, adafruit:SOT23-5L
- added L10: 15nH, Nordic_nRF:RESC0402_N
- added L8: 3.9nH, Nordic_nRF:RESC0402_N
- added L9: 10µH, Nordic_nRF:RESC0603_N
- added LDO1: AP2112-3.3K, tilesPartComp:SOT25
- added LED1: Orange, adafruit:CHIP-LED0603
- added MOS1: DMG3415U-7, tilesPartComp:SOT23
- added U$1: ZX62R-B-5P(30), tilesPartComp:ZX62R-B-5P(30)
- added U$7: CP2102N-A01-GQFN24, tilesPartComp:QFN-24
- added X5: 32MHz, Nordic_nRF:BT-XTAL_2016_N
- added X6: 32.768kHz, Nordic_nRF:XTAL_3215_N
- C1, C2: value 22pF -> 10µF; device microbuilder:0603-NO -> rcl:C0402K
- C3: value 10uF -> 10µF; device microbuilder:0805-NO -> rcl:C0402K
- C4: value 1uF -> 0.1µF; device microbuilder:0603-NO -> rcl:C0402K
- C5: value 10µF -> 4.7µF; device microbuilder:0805-NO -> rcl:C0402K
- D1: value RED -> NRVB120VLSF; device microbuilder:CHIPLED_0805_NOOUTLINE -> tilesPartComp:SOD123FL
- R1, R2: value 1K -> 100K; device microbuilder:0603-NO -> rcl:R0805
- R3: device microbuilder:0603-NO -> rcl:R0805
- R4: value 806K -> 10K; device microbuilder:0603-NO -> rcl:R0805
- R5: value 100K -> 1K; device microbuilder:0603-NO -> rcl:R0805
- U4: value CP2104 -> NRF52832; device microbuilder:QFN24_4MM_SMSC -> Nordic_nRF:QFN40P600X600X90-48_N
- moved R5 140.1 mm to (-31.8, -73.7)
- moved C4 132.3 mm to (-30.5, -63.5)
- moved C5 130.5 mm to (-30.5, -68.6)
- moved R4 124.6 mm to (-21.6, -58.4)
- moved R3 119.4 mm to (-21.6, -48.3)
- moved C3 116.1 mm to (-21.6, -53.3)
- moved C2 99.1 mm to (-1.27, -19.1)
- moved C1 93.3 mm to (-1.27, -15.2)
- moved R2 93.2 mm to (-1.27, -10.2)
- moved D1 91.2 mm to (0.00, -33.0)
- moved R1 85.1 mm to (-1.27, -3.81)
- moved U4 60.1 mm to (21.2, 16.2)
Connections:
- removed net 3.3V: C10.1, C3.1, C8.1, D4.C, MS1.2, MS1.3, R7.2, U1.11, U2.5, U4.5, U4.6, U4.7, X1.1
- removed net A0/0.02: MS1.5, U1.15
- removed net A1/0.03: MS1.6, U1.16
- removed net A2/0.04: MS1.7, U1.17
- removed net A3/0.05: MS1.8, U1.18
- removed net A4/0.28: MS1.9, U1.5
- removed net A5/0.29: MS1.10, U1.6
- removed net A6/P0.30: MS1.20, U1.7
- removed net A7/P0.31: C12.1, MS1.21, R4.2, R6.1, U1.8
- removed net DFU: MS1.16, SW2.B, SW2.B', U1.34
- removed net EN: MS1.27, R5.1, U2.3
- removed net FRST: TP2.P$1, U1.38
- removed net LED1: R1.2, U1.31
- removed net LED2: R2.2, U1.33
- removed net MISO: MS1.13, U1.28
- removed net MOSI: MS1.12, U1.27
- removed net N$11: R9.1, U4.21
- removed net N$13: C11.1, SJ2.2
- removed net N$14: C7.1, U4.16
- removed net N$7: D2.A, R2.1
- removed net P0.09/NFC1: C13.1, JP2.1, U1.22
- removed net P0.10/NFC2: C9.1, JP1.1, U1.23
- removed net RESET: D4.A, MS1.1, R7.1, SJ2.1, SW1.A, SW1.A', U1.35, X1.10
- removed net SCK: MS1.11, U1.26
- removed net SCL: MS1.18, U1.3
- removed net SDA: MS1.17, U1.2
- removed net SWCLK: TP4.P$1, U1.36, X1.4
- removed net SWO: U1.32, X1.6
- removed net VBUS: CHG.A, D5.A, MS1.26, Q3.1, R12.2, U3.4, U4.8, X3.VBUS
- removed net VIN: C6.1, D5.C, Q3.2, R5.2, U2.1
- new net ANT3: C35.1, L8.1, U4.30
- new net DEC1: C36.1, U4.1
- new net DEC2: C38.1, U4.32
- new net DEC3: C39.1, U4.33
- new net DEC4: C42.1, L10.2, U4.46
- new net GND@EXP: U$7.EXP
- new net N$6: IC1.5, R4.1
- new net P0.00/XL1: C43.2, U4.2, X6.1
- new net P0.01: U4.11
- new net P0.01/XL2: C44.2, U4.3, X6.2
- new net P0.02: U4.4
- new net P0.03: U4.5
- new net P0.04: U4.6
- new net P0.05: U4.7
- new net P0.09: U4.12
- new net P0.12: U4.15
- new net P0.13: U4.16
- new net P0.14: U4.17
- new net P0.17: U4.20
- new net P0.18/SWO: U4.21
- new net P0.19: U4.22
- new net P0.20: U4.23
- new net P0.21/RESET: U4.24
- new net P0.22: U4.27
- new net P0.23: U4.28
- new net P0.24: U4.29
- new net P0.25: U4.37
- new net P0.26: U4.38
- new net P0.28: U4.40
- new net P0.29: U4.41
- new net P0.30: U4.42
- new net P0.31: U4.43
- new net RF: L8.2
- new net SWDCLK: U4.25
- new net V+: C1.1, C37.1, C4.1, C40.1, C41.1, C5.1, LDO1.5, R5.2, U$7.5, U$7.6, U$7.7, U4.13, U4.36, U4.48
- new net X3: C34.1, U4.34, X5.1
- net DTR: now also U$7.23; no longer C11.2, U4.23
- net GND: now also C33.2, C34.2, C35.2, C36.2, C37.2, C38.2, C39.2, C40.2, C41.2, C42.2, C43.1, C44.1, IC1.2, LDO1.2, R2.2, R4.2, U$1.5, U$7.2, U4.31, U4.45, U4.PAD, U4.PAD@VIA01, U4.PAD@VIA02, U4.PAD@VIA03, U4.PAD@VIA04, U4.PAD@VIA05, U4.PAD@VIA06, U4.PAD@VIA07, U4.PAD@VIA08, U4.PAD@VIA09, U4.PAD@VIA10, U4.PAD@VIA11, U4.PAD@VIA12, U4.PAD@VIA13, U4.PAD@VIA14, U4.PAD@VIA15, U4.PAD@VIA16, X5.2, X5.4; no longer C10.2, C12.2, C13.2, C6.2, C7.2, C8.2, C9.2, D1.C, D2.C, MS1.4, R12.1, R6.2, R8.2, SW1.B, SW1.B', SW2.A, SW2.A', U1.1, U1.12, U1.24, U1.39, U2.2, U3.2, U4.2, U4.THERM, X1.3, X1.5, X1.7, X1.9, X2.1, X3.BASE@1, X3.BASE@2, X3.GND, X3.SPRT@1, X3.SPRT@2, X3.SPRT@3, X3.SPRT@4
- net N$1: now also LDO1.3, R1.1; no longer C1.1, U1.13, X4.P$1
- net N$10: now also L9.1, U4.47; no longer R8.1, U3.5
- net N$2: now also D1.C, LDO1.1, MOS1.2, R1.2; no longer U1.14, X4.P$2
- net N$3: now also IC1.1, R3.2; no longer L2.2, U1.10
- net N$4: now also LED1.C; no longer CHG.C
- net N$5: now also R5.1, U$7.9; no longer D1.A, R1.1
- net N$8: now also C33.1, U4.35, X5.3; no longer C4.1, L2.1, U1.9
- net N$9: now also L10.1, L9.2; no longer R3.2, U3.1
- net P0.07: now also U4.9; no longer MS1.23, U1.20
- net P0.11: now also U4.14; no longer MS1.22, U1.25
- net P0.15: now also U4.18; no longer MS1.24, U1.29
- net P0.16: now also U4.19; no longer MS1.25, U1.30
- net P0.27: now also U4.39; no longer MS1.19, U1.4
- net RXD: now also U$7.20, U4.10; no longer MS1.14, R9.2, U1.21
- net SWDIO: now also U4.26; no longer TP3.P$1, U1.37, X1.2
- net TXD: now also U$7.21, U4.8; no longer MS1.15, U1.19, U4.20
- net USBD+: now also U$1.2, U$7.3; no longer U4.3, X3.D+
- net USBD-: now also U$1.3, U$7.4; no longer U4.4, X3.D-
- net VBAT: now also C3.1, D1.A, IC1.3, IC1.4, LED1.A, MOS1.1, MOS1.3, R2.1, U$1.1, U$7.8; no longer C5.1, MS1.28, Q3.3, R4.1, U3.3, X2.2
Routing:
- net GND: track 0.00 -> 26.9 mm, vias 0 -> 23
- net V+: track 0.00 -> 24.1 mm, vias 0 -> 3
- net P0.00/XL1: track 0.00 -> 9.18 mm
- net X3: track 0.00 -> 8.06 mm
- net P0.01/XL2: track 0.00 -> 7.69 mm
- net TXD: track 0.00 -> 7.50 mm
- net RXD: track 0.00 -> 7.50 mm
- net P0.09: track 0.00 -> 7.50 mm
- net P0.07: track 0.00 -> 7.50 mm
- net P0.05: track 0.00 -> 7.50 mm
- net P0.04: track 0.00 -> 7.50 mm
- net P0.03: track 0.00 -> 7.50 mm
- net P0.02: track 0.00 -> 7.50 mm
- net P0.01: track 0.00 -> 7.50 mm
- net P0.24: track 0.00 -> 6.27 mm
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- added copper zone on layer 1, net GND
- added copper zone on layer 16, net GND

Commit message: ADD: microbuilder lib
Parts:
- added ANT2: (no value), tilesPartComp:2450AT45A100
- added B1: (no value), microbuilder:BTN_KMR2_4.6X2.8
- added C6, C7: 0.1µF, rcl:C0402K
- added C9: 1.5pF, rcl:C0805
- added D2: 1N4148, microbuilder:SOD-323
- added DFU, FRST: (no value), microbuilder:TESTPOINT_ROUND_2MM
- added DSG, U$9: CSD16406Q3, tilesPartComp:VSON-CLIP-8
- added JTAG1: (no value), microbuilder:2X05_1.27MM_SMT
- added L3: 3.9nH, rcl:L2012C
- added L4: DNP, rcl:L2012C
- added R6: 10K, rcl:R0805
- added R7: 330, rcl:R0805
- added R8: 2.2K, rcl:R0805
- added SJ1: (no value), microbuilder:SOLDERJUMPER_CLOSEDWIRE
- added U$12: BQ297XY, tilesPartComp:WSON_6
- added U$14: GM351824, tilesPartComp:GM351824
Connections:
- new net N$11: DSG.5, DSG.6, DSG.7, DSG.8, DSG.EXP, U$9.5, U$9.6, U$9.7, U$9.8, U$9.EXP
- new net N$12: DSG.4, U$12.3
- new net N$13: C7.1, R7.2, U$12.5
- new net N$14: U$12.2, U$9.4
- new net N$15: R8.1, U$12.6
- new net N$16: C7.2, DSG.1, DSG.2, DSG.3, U$12.4, U$14.-
- new net N$19: ANT2.1, C9.2, L3.1
- new net N$7: C6.2, SJ1.1
- net DTR: now also C6.1
- net GND: now also B1.B, B1.B', JTAG1.3, JTAG1.5, JTAG1.7, JTAG1.9, L3.2, L4.2, R8.2, U$9.1, U$9.2, U$9.3
- net P0.18/SWO: now also JTAG1.6
- net P0.20: now also DFU.P$1
- net P0.21/RESET: now also B1.A, B1.A', D2.A, JTAG1.10, R6.1, SJ1.2
- net P0.22: now also FRST.P$1
- net RF: now also C9.1, L4.1
- net SWDCLK: now also JTAG1.4
- net SWDIO: now also JTAG1.2
- net V+: now also D2.C, JTAG1.1, R6.2
- net VBAT: now also R7.1, U$14.+
Routing:
- net N$19: track 0.00 -> 4.40 mm
- net RF: track 0.95 -> 3.03 mm

Commit message: UPD: schematics
Parts:
- removed C35: 0.8pF, Nordic_nRF:RESC0402_N
- removed C9: 1.5pF, rcl:C0805
- removed L3: 3.9nH, rcl:L2012C
- removed L4: DNP, rcl:L2012C
- removed L8: 3.9nH, Nordic_nRF:RESC0402_N
- added C8: 0.1µF, rcl:C0603
- added F1: 2450FM07A0029, tilesPartComp:0402_RF
- added H1: HDC1080, tilesPartComp:PWSON_DMB
- added R10, R9: 10K, rcl:R0603
- added T1: SI7051-A20, tilesPartComp:DFN-6
- renumbered U$9 to CHG
Connections:
- removed net ANT3: C35.1, L8.1, U4.30
- removed net N$19: ANT2.1, C9.2, L3.1
- new net N$17: F1.1, U4.30
- new net VDD: C8.1, H1.5, R10.2, R9.2, T1.5
- net GND: now also C8.2, F1.GND@2, H1.2, T1.2; no longer C35.2, L3.2, L4.2
- net P0.25: now also H1.1, R9.1, T1.1
- net P0.26: now also H1.6, R10.1, T1.6
- net RF: now also ANT2.1, F1.3; no longer C9.1, L4.1, L8.2
Routing:
- net N$19: track 4.40 -> 0.00 mm
- net ANT3: track 3.39 -> 0.00 mm
- net RF: track 3.03 -> 0.00 mm
- net GND: track 26.9 -> 26.4 mm

Commit message: UPD: schem
Parts:
- removed R10: 10K, rcl:R0603
- removed X5: 32MHz, Nordic_nRF:BT-XTAL_2016_N
- added C9: 1nF, rcl:C0603
- added R11: 806K, rcl:R0603
- added R12: 2M, rcl:R0603
- added R15: 10K, rcl:R0603
- added X1: LFXTAL069526, tilesPartComp:1612
- C1, C2, C3: device rcl:C0402K -> rcl:C0805
- C38: value N.M. -> DNP
- C4, C5, C6, C7: device rcl:C0402K -> rcl:C0603
- D2: device microbuilder:SOD-323 -> tilesPartComp:SOD123
- LED1: device adafruit:CHIP-LED0603 -> microbuilder:CHIPLED_0805
- R1, R2, R4, R5, R6, R7, R8: device rcl:R0805 -> rcl:R0603
- R3: value 1K -> 200; device rcl:R0805 -> rcl:R0603
- moved C7 306.5 mm to (-0.85, -433.0)
- moved D2 297.0 mm to (-1.57, -394.9)
- moved C6 296.0 mm to (-0.85, -382.2)
- moved R7 289.0 mm to (-0.85, -420.3)
- moved R5 284.9 mm to (-0.85, -356.8)
- moved R6 278.4 mm to (-0.85, -369.5)
- moved C5 277.1 mm to (-0.85, -344.1)
- moved LED1 275.3 mm to (0.00, -317.7)
- moved R8 270.3 mm to (-0.85, -407.6)
- moved C4 269.6 mm to (-0.85, -331.4)
- moved C3 251.4 mm to (-0.95, -303.9)
- moved C1 250.6 mm to (-0.95, -265.8)
- moved R3 243.9 mm to (-0.85, -291.2)
- moved R1 236.6 mm to (-0.85, -240.4)
- moved C2 234.1 mm to (-0.95, -253.1)
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- renumbered ANT2 to ANT1, U$1 to USB1, U$12 to U12, U$7 to U7
Connections:
- net GND: now also C9.1, R12.1, X1.2, X1.4; no longer X5.2, X5.4
- net N$8: now also X1.3; no longer X5.3
- net P0.25: now also R15.1; no longer R9.1
- net P0.26: now also R9.1; no longer R10.1
- net P0.31: now also C9.2, R11.1, R12.2
- net VBAT: now also R11.2
- net VDD: now also R15.2; no longer R10.2
- net X3: now also X1.1; no longer X5.1
Routing:
- net GND: track 26.4 -> 25.0 mm

Commit message: UPD: leds
Parts:
- added R10, R14: 5, rcl:R0603
- added R13: 65, rcl:R0603
- added RGB1: 150080M153000, tilesPartComp:RGBLED_0805
- ANT1: value (none) -> 2450AT45A100
- C4, C6, C7, C8: device rcl:C0603 -> rcl:C0603K
- moved C8 341.5 mm to (-0.88, -483.8)
- moved F1 259.7 mm to (50.7, 59.4), turned to 90 degrees
- moved C4 127.0 mm to (-0.88, -458.4)
- moved C6 88.9 mm to (-0.88, -471.1)
- moved C37 53.7 mm to (54.7, 51.4), turned to 270 degrees
- moved U4 48.2 mm to (50.6, 54.3), turned to 90 degrees
- moved C38 46.8 mm to (48.3, 60.1), turned to 90 degrees
- moved C39 45.5 mm to (47.3, 60.1), turned to 90 degrees
- moved C44 44.5 mm to (47.7, 44.0), turned to 0 degrees
- moved C36 44.4 mm to (48.2, 49.7), turned to 270 degrees
- moved C34 44.0 mm to (45.4, 62.1), turned to 0 degrees
- moved X6 43.2 mm to (47.0, 45.7), turned to 0 degrees
- moved C41 42.6 mm to (46.9, 49.7), turned to 270 degrees
- moved C33 42.1 mm to (45.4, 58.1), turned to 180 degrees
- moved C40 41.7 mm to (45.4, 57.1), turned to 180 degrees
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Connections:
- removed net GND@EXP: U7.EXP
- removed net VDD: C8.1, H1.5, R15.2, R9.2, T1.5
- new net N$19: R13.2, RGB1.1
- new net N$20: R10.2, RGB1.2
- new net N$21: R14.2, RGB1.3
- new net N$22: R14.1
- new net N$24: R10.1
- new net P0.06: R13.1
- new net VUSB: D1.A, IC1.4, LED1.A, MOS1.1, R2.1, U7.8, USB1.1
- net GND: now also F1.GND@4, U7.EXP
- net V+: now also C8.1, H1.5, R15.2, R9.2, RGB1.4, T1.5
- net VBAT: no longer D1.A, IC1.4, LED1.A, MOS1.1, R2.1, U7.8, USB1.1
Routing:
- net GND: track 25.0 -> 23.2 mm
- added copper zone on layer 16, net N$18
- removed copper zone on layer 16, net GND

Commit message: UPD: board
Parts:
- R10, R14: value 5 -> 22
- R13: value 65 -> 100
- moved R10 581.6 mm to (95.2, 50.8)
- moved R13 581.6 mm to (95.2, 45.7)
- moved R14 581.6 mm to (95.2, 40.6)
- moved RGB1 581.6 mm to (96.5, 55.9)
- moved C5 369.9 mm to (91.9, 14.0)
- moved LED1 369.9 mm to (92.7, 40.5)
- moved R3 369.9 mm to (91.9, 66.9)
- moved R5 369.9 mm to (91.9, 1.31)
- moved C3 329.6 mm to (44.8, 22.5), turned to 270 degrees
- moved X1 316.9 mm to (46.2, 60.1), turned to 270 degrees
- moved R4 305.3 mm to (36.8, 24.4), turned to 180 degrees
- moved R9 304.6 mm to (33.0, 57.1), turned to 180 degrees
- moved C2 302.2 mm to (66.4, 41.5)
- moved R15 297.9 mm to (33.0, 54.6), turned to 180 degrees
- moved C1 289.7 mm to (38.4, 21.2)
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Connections:
- removed net N$22: R14.1
- removed net N$24: R10.1
- removed net P0.06: R13.1
- net P0.02: now also R13.1
- net P0.03: now also R10.1
- net P0.04: now also R14.1
Routing:
- net VUSB: track 0.00 -> 24.6 mm
- net RF: track 0.00 -> 9.28 mm
- net TXD: track 7.50 -> 0.00 mm
- net RXD: track 7.50 -> 0.00 mm
- net P0.09: track 7.50 -> 0.00 mm
- net P0.07: track 7.50 -> 0.00 mm
- net P0.05: track 7.50 -> 0.00 mm
- net P0.04: track 7.50 -> 0.00 mm
- net P0.03: track 7.50 -> 0.00 mm
- net P0.02: track 7.50 -> 0.00 mm
- net P0.01: track 7.50 -> 0.00 mm
- net P0.24: track 6.27 -> 0.00 mm
- net VBAT: track 0.00 -> 6.19 mm
- net P0.23: track 5.59 -> 0.00 mm
- net P0.22: track 4.91 -> 0.00 mm
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- added copper zone on layer 16, net GND
- removed copper zone on layer 16, net N$18

Commit message: UPD: wiring
Parts:
- moved C6 540.4 mm to (64.0, 65.4), turned to 180 degrees
- moved C8 507.5 mm to (45.3, 21.6), turned to 180 degrees
- moved C4 483.5 mm to (45.3, 22.8), turned to 180 degrees
- moved C7 469.5 mm to (28.8, 22.8), turned to 180 degrees
- moved D2 461.9 mm to (63.1, 62.4), turned to 90 degrees
- moved R7 440.5 mm to (29.6, 19.1)
- moved R6 435.6 mm to (59.7, 61.8), turned to 270 degrees
- moved R8 425.2 mm to (30.1, 16.5), turned to 180 degrees
- moved R12 300.0 mm to (46.2, 54.4), turned to 270 degrees
- moved C9 286.5 mm to (42.8, 51.6)
- moved R11 278.3 mm to (39.4, 38.1)
- moved DFU 217.4 mm to (57.0, 61.7)
- moved FRST 212.5 mm to (53.8, 61.7)
- moved U12 196.0 mm to (34.3, 20.3), turned to 90 degrees
- moved DSG 195.6 mm to (29.2, 25.4)
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Routing:
- net P0.26: track 0.00 -> 46.4 mm, vias 0 -> 2
- net P0.25: track 0.00 -> 43.8 mm, vias 0 -> 2
- net V+: track 25.6 -> 50.0 mm
- net P0.21/RESET: track 0.00 -> 24.3 mm, vias 0 -> 3
- net DTR: track 0.00 -> 23.2 mm, vias 0 -> 2
- net SWDIO: track 0.00 -> 16.1 mm
- net TXD: track 0.00 -> 9.77 mm
- net P0.20: track 0.00 -> 9.68 mm, vias 0 -> 2
- net RXD: track 0.00 -> 9.51 mm
- net SWDCLK: track 0.20 -> 9.58 mm
- net P0.04: track 0.00 -> 5.86 mm
- net P0.22: track 0.00 -> 5.61 mm
- net P0.31: track 0.00 -> 5.21 mm
- net P0.18/SWO: track 0.00 -> 4.51 mm, vias 0 -> 2
- net P0.03: track 0.00 -> 4.25 mm
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
Commit message: UPD: finished wiring
Parts:
- added C10: 0.1µF, rcl:C0603K
- moved U$14 36.8 mm to (52.1, 39.0), flipped to the bottom, turned to 180 degrees
- moved R8 33.5 mm to (52.2, 41.7), turned to 270 degrees
- moved R7 30.2 mm to (49.9, 41.4), turned to 90 degrees
- moved U12 27.8 mm to (49.0, 43.9), turned to 180 degrees
- moved C7 26.8 mm to (48.1, 41.4), turned to 270 degrees
- moved LDO1 24.2 mm to (61.0, 35.1), turned to 90 degrees
- moved C4 23.6 mm to (57.8, 42.8), turned to 270 degrees
- moved DSG 22.5 mm to (45.0, 41.4), turned to 90 degrees
- moved CHG 21.5 mm to (45.0, 44.1), turned to 90 degrees
- moved C1 19.2 mm to (60.1, 39.2), turned to 90 degrees
- moved T1 18.2 mm to (57.7, 28.3)
- moved R1 18.0 mm to (57.5, 34.2), turned to 90 degrees
- moved C8 16.9 mm to (61.2, 27.3), turned to 0 degrees
- moved C2 11.7 mm to (57.5, 37.9), turned to 90 degrees
- moved LED1 10.6 mm to (50.8, 36.1), turned to 0 degrees
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Connections:
- net GND: now also C10.2
- net V+: now also C10.1
Routing:
- net V+: track 50.0 -> 120.5 mm, vias 3 -> 4
- net N$16: track 0.00 -> 46.2 mm, vias 0 -> 1
- net VBAT: track 6.19 -> 47.9 mm, vias 0 -> 1
- net USBD+: track 0.00 -> 29.9 mm, vias 0 -> 2
- net USBD-: track 0.00 -> 29.4 mm, vias 0 -> 2
- net P0.25: track 43.8 -> 58.1 mm, vias 2 -> 3
- net N$11: track 0.00 -> 11.7 mm
- net P0.31: track 5.21 -> 16.5 mm
- net P0.26: track 46.4 -> 57.4 mm, vias 2 -> 3
- net GND: track 24.0 -> 34.8 mm, vias 2 -> 80
- net N$4: track 0.00 -> 9.91 mm
- net VUSB: track 24.6 -> 32.6 mm, vias 0 -> 2
- net N$2: track 3.89 -> 8.76 mm
- net N$12: track 0.00 -> 3.98 mm
- net N$14: track 0.00 -> 3.71 mm
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Other:
- board size 100 x 80 mm -> 37.2 x 57.6 mm
