File: mcu.sch (EAGLE design)
At the start: 50 parts, among them Q3 DMG3415U-7, SW1 KMR2, SW2 KMR2, U1 MDBT42, U2 AP2112(3.3V), U3 MCP73831T-2ACI/OT, U4 CP2104, U5 MDBT42, X1 4u20317, X2 JSTPH, X3 4u20329, X4 32.768

Commit message: ADD: component and library
Parts:
- removed C10, C11: 0.1uF, microbuilder:CAP_CERAMIC0603_NO
- removed C12: 1nF, microbuilder:CAP_CERAMIC0603_NO
- removed C13, C9: 300pF, microbuilder:CAP_CERAMIC_0603MP
- removed C6, C8: 10µF, microbuilder:CAP_CERAMIC0805-NOOUTLINE
- removed C7: 10uf, microbuilder:CAP_CERAMIC0805-NOOUTLINE
- removed CHG: ORANGE, microbuilder:LED0805_NOOUTLINE
- removed D2: BLUE, microbuilder:LED0805_NOOUTLINE
- removed D4: 1N4148, microbuilder:DIODESOD-323
- removed D5: MBR120, microbuilder:DIODE-SCHOTTKYSOD-123
- removed FID1, FID3: FIDUCIAL_1MM, microbuilder:FIDUCIAL_1MM
- removed JP1, JP2: (no value), microbuilder:HEADER-1X12MM
- removed L2: 10uH, microbuilder:INDUCTOR0805-NO
- removed MS1: FEATHERWING_NODIM, microbuilder:FEATHERWING_NODIM
- removed Q3: DMG3415U-7, microbuilder:MOSFET-P
- removed R12: 100k, microbuilder:RESISTOR_0603_NOOUT
- removed R6: 2M, microbuilder:RESISTOR_0603_NOOUT
- removed R7, R8: 10K, microbuilder:RESISTOR_0603_NOOUT
- removed R9: 1K, microbuilder:RESISTOR_0603_NOOUT
- removed SJ2: BAT, microbuilder:SOLDERJUMPERCLOSED
- removed SW1, SW2: KMR2, microbuilder:SWITCH_TACT_SMT4.6X2.8
- removed TP2: FRST, microbuilder:TESTPOINT1.5X2.0MM_NOCREAM
- removed TP3, TP4: (no value), microbuilder:TESTPOINTROUND2MM
- removed U1, U5: MDBT42, microbuilder:NRF52832_MODULE_MDBT42
- removed U2: AP2112(3.3V), microbuilder:VREG_SOT23-5
- removed U3: MCP73831T-2ACI/OT, microbuilder:MCP73831/2
- removed X1: 4u20317, microbuilder:JTAG-CORTEXBOXPOSTS
- removed X2: JSTPH, microbuilder:CON_JST_PH_2PIN
- removed X3: 4u20329, microbuilder:USB_MICRO_20329_V2
- removed X4: 32.768, adafruit2:XTAL-3.2X1.5
- added C33, C34, C43, C44: 12pF, Nordic_nRF:CAPACITOR_0402_N
- added C35: 0.8pF, Nordic_nRF:CAPACITOR_0402_N
- added C36, C37, C40: 100nF, Nordic_nRF:CAPACITOR_0402_N
- added C38: N.M., Nordic_nRF:CAPACITOR_0402_N
- added C39: 100pF, Nordic_nRF:CAPACITOR_0402_N
- added C41: 4.7µF, Nordic_nRF:CAPACITOR_0603_N
- added C42: 1.0µF, Nordic_nRF:CAPACITOR_0603_N
- added IC1: MCP73831/OT, adafruit:MCP73831/OT
- added L10: 15nH, Nordic_nRF:INDUCTOR_0402_N
- added L8: 3.9nH, Nordic_nRF:INDUCTOR_0402_N
- added L9: 10µH, Nordic_nRF:INDUCTOR_0603_N
- added LDO1: AP2112-3.3K, tilesPartComp:AP2112-3.3K
- added LED1: Orange, adafruit:LEDCHIP-LED0603
- added MOS1: DMG3415U-7, tilesPartComp:DMG3415U-7
- added U$1: ZX62R-B-5P(30), tilesPartComp:ZX62R-B-5P(30)
- added U$7: CP2102N-A01-GQFN24, tilesPartComp:CP2102N-A01-GQFN24
- added X5: 32MHz, Nordic_nRF:XTAL_32MHZ
- added X6: 32.768kHz, Nordic_nRF:XTAL_32KHZ
- C1, C2: value 22pF -> 10µF; device microbuilder:CAP_CERAMIC0603_NO -> rcl:C-EUC0402K
- C3: value 10uF -> 10µF; device microbuilder:CAP_CERAMIC0805-NOOUTLINE -> rcl:C-EUC0402K
- C4: value 1uF -> 0.1µF; device microbuilder:CAP_CERAMIC0603_NO -> rcl:C-EUC0402K
- C5: value 10µF -> 4.7µF; device microbuilder:CAP_CERAMIC0805-NOOUTLINE -> rcl:C-EUC0402K
- D1: value RED -> NRVB120VLSF; device microbuilder:LED0805_NOOUTLINE -> tilesPartComp:NRVB120VLSF
- R1, R2: value 1K -> 100K; device microbuilder:RESISTOR_0603_NOOUT -> rcl:R-EU_R0805
- R3: device microbuilder:RESISTOR_0603_NOOUT -> rcl:R-EU_R0805
- R4: value 806K -> 10K; device microbuilder:RESISTOR_0603_NOOUT -> rcl:R-EU_R0805
- R5: value 100K -> 1K; device microbuilder:RESISTOR_0603_NOOUT -> rcl:R-EU_R0805
- U4: value CP2104 -> NRF52832; device microbuilder:CP2104 -> Nordic_nRF:NRF52832
Connections:
- removed net 3.3V: C10.1, C3.1, C8.1, D4.C, MS1.3V, MS1.AREF, R7.2, U1.VDD, U2.OUT, U4G$1.REGIN, U4G$1.VDD, U4G$1.VIO, X1.VCC
- removed net A0/0.02: MS1.GPIOA0, U1.P0.02/AIN0
- removed net A1/0.03: MS1.GPIOA1, U1.P0.03/AIN1
- removed net A2/0.04: MS1.GPIOA2, U1.P0.04/AIN2
- removed net A3/0.05: MS1.GPIOA3, U1.P0.05/AIN3
- removed net A4/0.28: MS1.GPIOA4, U1.P0.28/AIN4
- removed net A5/0.29: MS1.GPIOA5, U1.P0.29/AIN5
- removed net A6/P0.30: MS1.GPIO6, U1.P0.30/AIN6
- removed net A7/P0.31: C12.1, MS1.GPIO9, R4.2, R6.1, U1.P0.31/AIN7
- removed net DFU: MS1.NC, SW2.S, SW2.S1, U1.P0.20
- removed net EN: MS1.EN, R5.1, U2.EN
- removed net FRST: TP2.P$1, U1.P0.22
- removed net LED1: R1.2, U1.P0.17
- removed net LED2: R2.2, U1.P0.19
- removed net MISO: MS1.GPIOMISO, U1.P0.14
- removed net MOSI: MS1.GPIOMOSI, U1.P0.13
- removed net N$11: R9.1, U4G$1.TXD
- removed net N$13: C11.1, SJ2.2
- removed net N$14: C7.1, U4G$1.VPP
- removed net N$7: D2.A, R2.1
- removed net P0.09/NFC1: C13.1, JP2.1, U1.P0.09
- removed net P0.10/NFC2: C9.1, JP1.1, U1.P0.10
- removed net RESET: D4.A, MS1.!RESET, R7.1, SJ2.1, SW1.P, SW1.P1, U1.P0.21/RESET, X1.NRESET
- removed net SCK: MS1.GPIOSCK, U1.P0.12
- removed net SCL: MS1.GPIOSCL, U1.P0.26
- removed net SDA: MS1.GPIOSDA, U1.P0.25
- removed net SWCLK: TP4.P$1, U1.SWDCLK, X1.SWDCLK
- removed net SWO: U1.P0.18/SWO, X1.SWO
- removed net VBUS: CHG.A, D5.A, MS1.USB, Q3.G, R12.2, U3.VDD, U4G$1.VBUS, X3.VBUS
- removed net VIN: C6.1, D5.C, Q3.S, R5.2, U2.IN
- new net ANT3: C35.1, L8.1, U4.ANT@30
- new net DEC1: C36.1, U4.DEC1@01
- new net DEC2: C38.1, U4.DEC2@32
- new net DEC3: C39.1, U4.DEC3@33
- new net DEC4: C42.1, L10.2, U4.DEC4@46
- new net GND@EXP: U$7.GND@EXP
- new net N$6: IC1.PROG, R4.1
- new net P0.00/XL1: C43.2, U4.P0.00/XL1@02, X6.1
- new net P0.01: U4.P0.09/NFC1@11
- new net P0.01/XL2: C44.2, U4.P0.01/XL2@03, X6.2
- new net P0.02: U4.P0.02/AIN0@04
- new net P0.03: U4.P0.03/AIN1@05
- new net P0.04: U4.P0.04/AIN2@06
- new net P0.05: U4.P0.05/AIN3@07
- new net P0.09: U4.P0.10/NFC2@12
- new net P0.12: U4.P0.12@15
- new net P0.13: U4.P0.13@16
- new net P0.14: U4.P0.14@17
- new net P0.17: U4.P0.17@20
- new net P0.18/SWO: U4.P0.18/SWO@21
- new net P0.19: U4.P0.19@22
- new net P0.20: U4.P0.20@23
- new net P0.21/RESET: U4.P0.21/RESET@24
- new net P0.22: U4.P0.22@27
- new net P0.23: U4.P0.23@28
- new net P0.24: U4.P0.24@29
- new net P0.25: U4.P0.25@37
- new net P0.26: U4.P0.26@38
- new net P0.28: U4.P0.28@40
- new net P0.29: U4.P0.29@41
- new net P0.30: U4.P0.30@42
- new net P0.31: U4.P0.31@43
- new net RF: L8.2
- new net SWDCLK: U4.SWDCLK@25
- new net V+: C1.1, C37.1, C4.1, C40.1, C41.1, C5.1, LDO1.VOUT, R5.2, U$7.VDD, U$7.VIO, U$7.VREGIN, U4.VDD@13, U4.VDD@36, U4.VDD@48
- new net X3: C34.1, U4.XC1@34, X5.1
- net DTR: now also U$7.DTR; no longer C11.2, U4G$1.DTR
- net GND: now also C33.2, C34.2, C35.2, C36.2, C37.2, C38.2, C39.2, C40.2, C41.2, C42.2, C43.1, C44.1, IC1.VSS, LDO1.GND, R2.2, R4.2, U$1.5, U$7.GND, U4.VSS@31, U4.VSS@45, X5.2, X5.4; no longer C10.2, C12.2, C13.2, C6.2, C7.2, C8.2, C9.2, D1.C, D2.C, MS1.GND, R12.1, R6.2, R8.2, SW1.S, SW1.S1, SW2.P, SW2.P1, U1.GND@1, U1.GND@2, U1.GND@3, U1.GND@4, U2.GND, U3.VSS, U4G$1.GND, U4G$2.TP, X1.GND@1, X1.GND@2, X1.GNDDETECT, X1.KEY, X2.1, X3.GND
- net N$1: now also LDO1.EN, R1.1; no longer C1.1, U1.P0.00/XL1, X4.P$1
- net N$10: now also L9.1, U4.DCC@47; no longer R8.1, U3.PROG
- net N$2: now also D1.C, LDO1.VIN, MOS1.S, R1.2; no longer U1.P0.01/XL2, X4.P$2
- net N$3: now also IC1.STAT, R3.2; no longer L2.2, U1.DCC
- net N$4: now also LED1.C; no longer CHG.C
- net N$5: now also R5.1, U$7.!RSTB; no longer D1.A, R1.1
- net N$8: now also C33.1, U4.XC2@35, X5.3; no longer C4.1, L2.1, U1.DEC4
- net N$9: now also L10.1, L9.2; no longer R3.2, U3.STAT
- net P0.07: now also U4.P0.07@09; no longer MS1.GPIO11, U1.P0.07
- net P0.11: now also U4.P0.11@14; no longer MS1.GPIO10, U1.P0.11
- net P0.15: now also U4.P0.15@18; no longer MS1.GPIO12, U1.P0.15
- net P0.16: now also U4.P0.16@19; no longer MS1.GPIO13, U1.P0.16
- net P0.27: now also U4.P0.27@39; no longer MS1.GPIO5, U1.P0.27
- net RXD: now also U$7.RXD, U4.P0.08@10; no longer MS1.GPIORX, R9.2, U1.P0.08
- net SWDIO: now also U4.SWDIO@26; no longer TP3.P$1, U1.SWDIO, X1.SWDIO
- net TXD: now also U$7.TXD, U4.P0.06@08; no longer MS1.GPIOTX, U1.P0.06, U4G$1.RXD
- net USBD+: now also U$1.2, U$7.D+; no longer U4G$1.D+, X3.D+
- net USBD-: now also U$1.3, U$7.D-; no longer U4G$1.D-, X3.D-
- net VBAT: now also C3.1, D1.A, IC1.VBAT, IC1.VDD, LED1.A, MOS1.D, MOS1.G, R2.1, U$1.1, U$7.VBUS; no longer C5.1, MS1.VBAT, Q3.D, R4.1, U3.VBAT, X2.2
Other:
- note added: "USB Power"
- note added: "Voltage Regulator"
- note added: "nFR52832 QFAA QFN48 with DC/DC regulator setup"
- note removed: "0.1uF+10K @ 3.3V = ~1.2ms to 0.7VCC"
- note removed: "1.0K = 1000mA"
- note removed: "10K = 100mA"
- note removed: "2.0K = 500mA"
- note removed: "5.0K = 200mA"
- note removed: "Adafruit Feather Pinout"
- note removed: "Dropout Voltage (25°C): 100mA: ~250/~40mV 300mA: ~300/~125mV 600mA: ~375/~260mV"
- note removed: "Dynamic VIN selection: VBUS (USB) will override VBAT (LIPO) via D5 when both are present."
- note removed: "JST PH LIPO INPUT"
- note removed: "LIPO CHARGING"
- note removed: "LIPO MONITORING"
- note removed: "POWER AND FILTERING (600mA Output)"
- note removed: "See: https://devzone.nordicsemi.com/blogs/943/measuring-lithium-battery-voltage-with-nrf52/ Maximum voltage: 4.2 V * (2 M/(0.8 M+2 M)) = 3 V Minimum voltage: 2.7 V * (2 M/(0.8 M+2 M)) = 1.93 V ADC value at 4.2 V - 12 bit setup: 3 V * (1/5) / 0.6 V * 4095 = 4095 ADC value at 2.7 V - 12 bit setup: 1.93 V * (1/5) / 0.6 V * 4095 = 2634 Usable ADC resolution - 12 bit setup: 4095 - 2634 = 1461"
- note removed: "To charge the LIPO, insert the battery in the JST PH connector and connect USB at the same time."
- note removed: "USB POWER"
- note removed: "USB RESET (DTR)"
- note removed: "USB/TTL Bridge"

Commit message: ADD: microbuilder lib
Parts:
- added ANT2: (no value), tilesPartComp:2450AT45A100
- added B1: (no value), microbuilder:SWITCH_TACT_SMT4.6X2.8
- added C6, C7: 0.1µF, rcl:C-EUC0402K
- added C9: 1.5pF, rcl:C-EUC0805
- added D2: 1N4148, microbuilder:DIODESOD-323
- added DFU, FRST: (no value), microbuilder:TESTPOINTROUND2MM
- added DSG, U$9: CSD16406Q3, tilesPartComp:CSD16406Q3
- added JTAG1: (no value), microbuilder:JTAG-CORTEXM3
- added L3: 3.9nH, rcl:L-USL2012C
- added L4: DNP, rcl:L-USL2012C
- added R6: 10K, rcl:R-EU_R0805
- added R7: 330, rcl:R-EU_R0805
- added R8: 2.2K, rcl:R-EU_R0805
- added SJ1: (no value), microbuilder:SOLDERJUMPER_CLOSED
- added U$12: BQ297XY, tilesPartComp:BQ297XY
- added U$14: GM351824, tilesPartComp:GM351824
Connections:
- new net N$11: DSG.D, U$9.D
- new net N$12: DSG.G, U$12.DOUT
- new net N$13: C7.1, R7.2, U$12.BAT
- new net N$14: U$12.COUT, U$9.G
- new net N$15: R8.1, U$12.V-
- new net N$16: C7.2, DSG.S, U$12.VSS, U$14.-
- new net N$19: ANT2.1, C9.2, L3.1
- new net N$7: C6.2, SJ1.1
- net DTR: now also C6.1
- net GND: now also B1.S, B1.S1, JTAG1.3, JTAG1.5, JTAG1.7, JTAG1.9, L3.2, L4.2, R8.2, U$9.S
- net P0.18/SWO: now also JTAG1.6
- net P0.20: now also DFU.P$1
- net P0.21/RESET: now also B1.P, B1.P1, D2.A, JTAG1.10, R6.1, SJ1.2
- net P0.22: now also FRST.P$1
- net RF: now also C9.1, L4.1
- net SWDCLK: now also JTAG1.4
- net SWDIO: now also JTAG1.2
- net V+: now also D2.C, JTAG1.1, R6.2
- net VBAT: now also R7.1, U$14.+
Other:
- note added: "1.0K = 1000mA"
- note added: "10K = 100mA"
- note added: "2.0K = 500mA"
- note added: "20K = 50mA"
- note added: "5.0K = 200mA"
- note added: "Auto reset from USB signal"
- note added: "Battery protection"
- note added: "Check charge V based on battery type"
- note added: "Check what available"
- note added: "PIN_DFU / P0.20 = if GND at startup will go into bootloader FRST / P0.22 = if GND at startup factory reset and reboot into bootloader"
- note added: "R-PROG"
- note added: "Reset button"
- note added: "See datasheet for optimal positioning"
- note added: "TI bq2970, bq2971, bq2972, bq2973 depending on battery parameters"
- note added: "Testpoints"

Commit message: UPD: schematics
Parts:
- removed C35: 0.8pF, Nordic_nRF:CAPACITOR_0402_N
- removed C9: 1.5pF, rcl:C-EUC0805
- removed L3: 3.9nH, rcl:L-USL2012C
- removed L4: DNP, rcl:L-USL2012C
- removed L8: 3.9nH, Nordic_nRF:INDUCTOR_0402_N
- added C8: 0.1µF, rcl:C-EUC0603
- added F1: 2450FM07A0029, tilesPartComp:2450FM07A0029
- added H1: HDC1080, tilesPartComp:HDC1080
- added R10, R9: 10K, rcl:R-US_R0603
- added T1: SI7051-A20, tilesPartComp:SI7051-A20
- renumbered U$9 to CHG
Connections:
- removed net ANT3: C35.1, L8.1, U4.ANT@30
- removed net N$19: ANT2.1, C9.2, L3.1
- new net N$17: F1.IN, U4.ANT@30
- new net VDD: C8.1, H1.VDD, R10.2, R9.2, T1.VDD
- net GND: now also C8.2, F1.GND@2, H1.GND, T1.GND; no longer C35.2, L3.2, L4.2
- net P0.25: now also H1.SDA, R9.1, T1.SDA
- net P0.26: now also H1.SCL, R10.1, T1.SCL
- net RF: now also ANT2.1, F1.OUT; no longer C9.1, L4.1, L8.2
Other:
- note added: "Temperature and Humidity sensors"
- moved on the sheet: ANT2

Commit message: UPD: schem
Parts:
- removed R10: 10K, rcl:R-US_R0603
- removed X5: 32MHz, Nordic_nRF:XTAL_32MHZ
- added C9: 1nF, rcl:C-EUC0603
- added R11: 806K, rcl:R-EU_R0603
- added R12: 2M, rcl:R-EU_R0603
- added R15: 10K, rcl:R-EU_R0603
- added X1: LFXTAL069526, tilesPartComp:LFXTAL069526
- C1, C2, C3: device rcl:C-EUC0402K -> rcl:C-EUC0805
- C38: value N.M. -> DNP
- C4, C5, C6, C7: device rcl:C-EUC0402K -> rcl:C-EUC0603
- D2: device microbuilder:DIODESOD-323 -> tilesPartComp:1N4148W-7-F
- LED1: device adafruit:LEDCHIP-LED0603 -> microbuilder:LED0805
- R1, R2, R4, R5, R6, R7, R8: device rcl:R-EU_R0805 -> rcl:R-EU_R0603
- R3: value 1K -> 200; device rcl:R-EU_R0805 -> rcl:R-EU_R0603
- R9: device rcl:R-US_R0603 -> rcl:R-EU_R0603
- renumbered ANT2 to ANT1, U$1 to USB1, U$12 to U12, U$7 to U7
Connections:
- net GND: now also C9.1, R12.1, X1.GND@1, X1.GND@2; no longer X5.2, X5.4
- net N$8: now also X1.2; no longer X5.3
- net P0.25: now also R15.1; no longer R9.1
- net P0.26: now also R9.1; no longer R10.1
- net P0.31: now also C9.2, R11.1, R12.2
- net VBAT: now also R11.2
- net VDD: now also R15.2; no longer R10.2
- net X3: now also X1.1; no longer X5.1
Other:
- note added: "LIPO MONITORING"
- note added: "See: https://devzone.nordicsemi.com/blogs/943/measuring-lithium-battery-voltage-with-nrf52/ Maximum voltage: 4.2 V * (2 M/(0.8 M+2 M)) = 3 V Minimum voltage: 2.7 V * (2 M/(0.8 M+2 M)) = 1.93 V ADC value at 4.2 V - 12 bit setup: 3 V * (1/5) / 0.6 V * 4095 = 4095 ADC value at 2.7 V - 12 bit setup: 1.93 V * (1/5) / 0.6 V * 4095 = 2634 Usable ADC resolution - 12 bit setup: 4095 - 2634 = 1461"
- moved on the sheet: C33

Commit message: UPD: leds
Parts:
- added R10, R14: 5, rcl:R-EU_R0603
- added R13: 65, rcl:R-EU_R0603
- added RGB1: 150080M153000, tilesPartComp:150080M153000
- ANT1: value (none) -> 2450AT45A100
- C4, C6, C7, C8: device rcl:C-EUC0603 -> rcl:C-EUC0603K
Connections:
- removed net GND@EXP: U7.GND@EXP
- removed net VDD: C8.1, H1.VDD, R15.2, R9.2, T1.VDD
- new net N$19: R13.2, RGB1.R
- new net N$20: R10.2, RGB1.G
- new net N$21: R14.2, RGB1.B
- new net N$22: R14.1
- new net N$24: R10.1
- new net P0.06: R13.1
- new net VUSB: D1.A, IC1.VDD, LED1.A, MOS1.G, R2.1, U7.VBUS, USB1.1
- net GND: now also F1.GND@4, U7.GND@EXP
- net V+: now also C8.1, H1.VDD, R15.2, R9.2, RGB1.VDD, T1.VDD
- net VBAT: no longer D1.A, IC1.VDD, LED1.A, MOS1.G, R2.1, U7.VBUS, USB1.1

Commit message: UPD: board
Parts:
- R10, R14: value 5 -> 22
- R13: value 65 -> 100
Connections:
- removed net N$22: R14.1
- removed net N$24: R10.1
- removed net P0.06: R13.1
- net P0.02: now also R13.1
- net P0.03: now also R10.1
- net P0.04: now also R14.1
Changed lines of the file:
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@@
 <part name="RGB1" library="tilesPartComp" deviceset="150080M153000" device=""/>
 <part name="VDD_10" library="supply2" library_urn="urn:adsk.eagle:library:372" deviceset="V+" device="" value="3.3V"/>
-<part name="GND18" library="supply1" library_urn="urn:adsk.eagle:library:371" deviceset="GND" device=""/>
-<part name="R10" library="rcl" library_urn="urn:adsk.eagle:library:334" deviceset="R-EU_" device="R0603" package3d_urn="urn:adsk.eagle:package:23555/2" value="5"/>
-<part name="R13" library="rcl" library_urn="urn:adsk.eagle:library:334" deviceset="R-EU_" device="R0603" package3d_urn="urn:adsk.eagle:package:23555/2" value="65"/>
-<part name="R14" library="rcl" library_urn="urn:adsk.eagle:library:334" deviceset="R-EU_" device="R0603" package3d_urn="urn:adsk.eagle:package:23555/2" value="5"/>
+<part name="R10" library="rcl" library_urn="urn:adsk.eagle:library:334" deviceset="R-EU_" device="R0603" package3d_urn="urn:adsk.eagle:package:23555/2" value="22"/>
+<part name="R13" library="rcl" library_urn="urn:adsk.eagle:library:334" deviceset="R-EU_" device="R0603" package3d_urn="urn:adsk.eagle:package:23555/2" value="100"/>
+<part name="R14" library="rcl" library_urn="urn:adsk.eagle:library:334" deviceset="R-EU_" device="R0603" package3d_urn="urn:adsk.eagle:package:23555/2" value="22"/>
 </parts>
 <sheets>
@@
 <instance part="RGB1" gate="150080M153000-RGB-LED" x="-93.98" y="116.84"/>
 <instance part="VDD_10" gate="1" x="-81.28" y="132.08"/>
-<instance part="GND18" gate="1" x="-160.02" y="119.38"/>
 <instance part="R10" gate="G$1" x="-134.62" y="124.46"/>
 <instance part="R13" gate="G$1" x="-134.62" y="142.24"/>
@@
 <wire x1="254" y1="337.82" x2="254" y2="335.28" width="0.1524" layer="91"/>
 </segment>
-<segment>
-<pinref part="GND18" gate="1" pin="GND"/>
-<wire x1="-160.02" y1="124.46" x2="-160.02" y2="121.92" width="0.1524" layer="91"/>
-</segment>
 </net>
 <net name="DEC1" class="0">
@@
 <pinref part="U4" gate="U$1" pin="P0.02/AIN0@04"/>
 </segment>
+<segment>
+<pinref part="R13" gate="G$1" pin="1"/>
+<wire x1="-139.7" y1="142.24" x2="-144.78" y2="142.24" width="0.1524" layer="91"/>
+<label x="-144.78" y="142.24" size="1.778" layer="95" rot="R180" xref="yes"/>
+</segment>
 </net>
 <net name="P0.03" class="0">
@@
 <pinref part="U4" gate="U$1" pin="P0.03/AIN1@05"/>
 </segment>
+<segment>
+<pinref part="R10" gate="G$1" pin="1"/>
+<wire x1="-139.7" y1="124.46" x2="-144.78" y2="124.46" width="0.1524" layer="91"/>
+<label x="-144.78" y="124.46" size="1.778" layer="95" rot="R180" xref="yes"/>
+</segment>
 </net>
 <net name="P0.04" class="0">
@@
 <label x="35.56" y="228.6" size="1.27" layer="95" rot="R180" xref="yes"/>
 <pinref part="U4" gate="U$1" pin="P0.04/AIN2@06"/>
+</segment>
+<segment>
+<pinref part="R14" gate="G$1" pin="1"/>
+<wire x1="-139.7" y1="91.44" x2="-144.78" y2="91.44" width="0.1524" layer="91"/>
+<label x="-144.78" y="91.44" size="1.778" layer="95" rot="R180" xref="yes"/>
 </segment>
 </net>
@@
 </segment>
 </net>
-<net name="N$22" class="0">
-<segment>
-<pinref part="R14" gate="G$1" pin="1"/>
-<wire x1="-139.7" y1="91.44" x2="-144.78" y2="91.44" width="0.1524" layer="91"/>
-<label x="-144.78" y="91.44" size="1.778" layer="95" rot="R180" xref="yes"/>
-</segment>
-</net>
-<net name="P0.06" class="0">
-<segment>
-<pinref part="R13" gate="G$1" pin="1"/>
-<wire x1="-139.7" y1="142.24" x2="-144.78" y2="142.24" width="0.1524" layer="91"/>
-<label x="-144.78" y="142.24" size="1.778" layer="95" rot="R180" xref="yes"/>
-</segment>
-</net>
-<net name="N$24" class="0">
-<segment>
-<pinref part="R10" gate="G$1" pin="1"/>
-<wire x1="-139.7" y1="124.46" x2="-144.78" y2="124.46" width="0.1524" layer="91"/>
-<label x="-144.78" y="124.46" size="1.778" layer="95" rot="R180" xref="yes"/>
-</segment>
-</net>

Commit message: UPD: finished wiring
Parts:
- added C10: 0.1µF, rcl:C-EUC0603K
Connections:
- net GND: now also C10.2
- net V+: now also C10.1
Other:
- moved on the sheet: C8
Changed lines of the file:
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@@
 <part name="R13" library="rcl" library_urn="urn:adsk.eagle:library:334" deviceset="R-EU_" device="R0603" package3d_urn="urn:adsk.eagle:package:23555/2" value="100"/>
 <part name="R14" library="rcl" library_urn="urn:adsk.eagle:library:334" deviceset="R-EU_" device="R0603" package3d_urn="urn:adsk.eagle:package:23555/2" value="22"/>
+<part name="C10" library="rcl" library_urn="urn:adsk.eagle:library:334" deviceset="C-EU" device="C0603K" package3d_urn="urn:adsk.eagle:package:23680/2" value="0.1µF"/>
+<part name="GND18" library="supply1" deviceset="GND" device=""/>
 </parts>
 <sheets>
@@
 <instance part="F1" gate="2450FM07A0029" x="137.16" y="220.98"/>
 <instance part="T1" gate="SI7051-A20" x="10.16" y="137.16"/>
-<instance part="C8" gate="G$1" x="55.88" y="149.86"/>
+<instance part="C8" gate="G$1" x="40.64" y="129.54"/>
 <instance part="VDD_9" gate="1" x="48.26" y="162.56"/>
 <instance part="GND14" gate="1" x="-7.62" y="127" rot="MR0"/>
 <instance part="H1" gate="HDC1080" x="10.16" y="104.14"/>
 <instance part="GND15" gate="1" x="-7.62" y="91.44" rot="MR0"/>
-<instance part="GND16" gate="1" x="55.88" y="139.7" rot="MR0"/>
+<instance part="GND16" gate="1" x="40.64" y="119.38" rot="MR0"/>
 <instance part="U$9" gate="G$1" x="160.02" y="124.46"/>
 <instance part="GND17" gate="1" x="160.02" y="81.28"/>
@@
 <instance part="R13" gate="G$1" x="-134.62" y="142.24"/>
 <instance part="R14" gate="G$1" x="-134.62" y="91.44"/>
+<instance part="C10" gate="G$1" x="40.64" y="99.06"/>
+<instance part="GND18" gate="1" x="40.64" y="88.9" rot="MR0"/>
 </instances>
 <busses>
@@
 <pinref part="C8" gate="G$1" pin="2"/>
 <pinref part="GND16" gate="1" pin="GND"/>
-<wire x1="55.88" y1="144.78" x2="55.88" y2="142.24" width="0.1524" layer="91"/>
+<wire x1="40.64" y1="124.46" x2="40.64" y2="121.92" width="0.1524" layer="91"/>
 </segment>
 <segment>
@@
 <wire x1="243.84" y1="337.82" x2="254" y2="337.82" width="0.1524" layer="91"/>
 <wire x1="254" y1="337.82" x2="254" y2="335.28" width="0.1524" layer="91"/>
+</segment>
+<segment>
+<pinref part="C10" gate="G$1" pin="2"/>
+<pinref part="GND18" gate="1" pin="GND"/>
+<wire x1="40.64" y1="93.98" x2="40.64" y2="91.44" width="0.1524" layer="91"/>
 </segment>
 </net>
@@
 <pinref part="VDD_9" gate="1" pin="V+"/>
 <wire x1="48.26" y1="154.94" x2="48.26" y2="160.02" width="0.1524" layer="91"/>
+<wire x1="35.56" y1="154.94" x2="48.26" y2="154.94" width="0.1524" layer="91"/>
+<pinref part="R9" gate="G$1" pin="2"/>
+<junction x="35.56" y="154.94"/>
 <wire x1="-17.78" y1="154.94" x2="35.56" y2="154.94" width="0.1524" layer="91"/>
+<pinref part="R15" gate="G$1" pin="2"/>
 <pinref part="T1" gate="SI7051-A20" pin="VDD"/>
-<wire x1="35.56" y1="154.94" x2="48.26" y2="154.94" width="0.1524" layer="91"/>
-<wire x1="25.4" y1="137.16" x2="48.26" y2="137.16" width="0.1524" layer="91"/>
-<wire x1="48.26" y1="137.16" x2="48.26" y2="154.94" width="0.1524" layer="91"/>
+<wire x1="25.4" y1="137.16" x2="40.64" y2="137.16" width="0.1524" layer="91"/>
+<pinref part="H1" gate="HDC1080" pin="VDD"/>
+<wire x1="40.64" y1="137.16" x2="48.26" y2="137.16" width="0.1524" layer="91"/>
+<wire x1="25.4" y1="104.14" x2="40.64" y2="104.14" width="0.1524" layer="91"/>
+<wire x1="40.64" y1="104.14" x2="48.26" y2="104.14" width="0.1524" layer="91"/>
+<wire x1="48.26" y1="137.16" x2="48.26" y2="104.14" width="0.1524" layer="91"/>
+<wire x1="48.26" y1="154.94" x2="48.26" y2="137.16" width="0.1524" layer="91"/>
 <junction x="48.26" y="154.94"/>
-<pinref part="H1" gate="HDC1080" pin="VDD"/>
-<wire x1="25.4" y1="104.14" x2="48.26" y2="104.14" width="0.1524" layer="91"/>
-<wire x1="48.26" y1="137.16" x2="48.26" y2="104.14" width="0.1524" layer="91"/>
 <junction x="48.26" y="137.16"/>
 <pinref part="C8" gate="G$1" pin="1"/>
-<wire x1="48.26" y1="154.94" x2="55.88" y2="154.94" width="0.1524" layer="91"/>
-<wire x1="55.88" y1="154.94" x2="55.88" y2="152.4" width="0.1524" layer="91"/>
-<pinref part="R9" gate="G$1" pin="2"/>
-<junction x="35.56" y="154.94"/>
-<pinref part="R15" gate="G$1" pin="2"/>
-</segment>
-<segment>
+<wire x1="40.64" y1="137.16" x2="40.64" y2="132.08" width="0.1524" layer="91"/>
+<junction x="40.64" y="137.16"/>
+<pinref part="C10" gate="G$1" pin="1"/>
+<wire x1="40.64" y1="101.6" x2="40.64" y2="104.14" width="0.1524" layer="91"/>
+<junction x="40.64" y="104.14"/>
+</segment>
+<segment>
