File: mcu.sch (EAGLE design)
At the start: 67 parts, among them IC1 MCP73831/OT, T1 SI7051-A20, U12 BQ297XY, U4 NRF52832, U7 CP2102N-A01-GQFN24, X1 LFXTAL069526, X6 32.768kHz

Commit message: UPD: board, and RF line
Parts:
- removed VDD: (no value), microbuilder:TESTPOINTROUND2MM
- added R16: 0, rcl:R-EU_R0402
- added R17, R18: DNP, rcl:R-EU_R0402
Connections:
- new net N$18: ANT1.1, R16.2, R17.2
- net GND: now also R17.1, R18.1
- net RF: now also R16.1, R18.2; no longer ANT1.1
- net V+: no longer VDD.P$1
Other:
- moved on the sheet: ANT1
Changed lines of the file:
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@@
 <?xml version="1.0" encoding="utf-8"?>
 <!DOCTYPE eagle SYSTEM "eagle.dtd">
-<eagle version="8.5.1">
+<eagle version="8.5.2">
 <drawing>
 <settings>
@@
 <part name="SWDIO" library="microbuilder" deviceset="TESTPOINT" device="ROUND2MM"/>
 <part name="GND" library="microbuilder" deviceset="TESTPOINT" device="ROUND2MM"/>
-<part name="VDD" library="microbuilder" deviceset="TESTPOINT" device="ROUND2MM"/>
 <part name="SWO" library="microbuilder" deviceset="TESTPOINT" device="ROUND2MM"/>
-<part name="VDD_11" library="supply2" library_urn="urn:adsk.eagle:library:372" deviceset="V+" device="" value="3.3V"/>
+<part name="GND12" library="supply1" deviceset="GND" device=""/>
+<part name="R16" library="rcl" library_urn="urn:adsk.eagle:library:334" deviceset="R-EU_" device="R0402" package3d_urn="urn:adsk.eagle:package:23547/2" value="0"/>
+<part name="R17" library="rcl" library_urn="urn:adsk.eagle:library:334" deviceset="R-EU_" device="R0402" package3d_urn="urn:adsk.eagle:package:23547/2" value="DNP"/>
+<part name="R18" library="rcl" library_urn="urn:adsk.eagle:library:334" deviceset="R-EU_" device="R0402" package3d_urn="urn:adsk.eagle:package:23547/2" value="DNP"/>
 </parts>
 <sheets>
@@
 <instance part="U12" gate="BQ297XY" x="-96.52" y="233.68"/>
 <instance part="U$14" gate="G$1" x="-40.64" y="233.68" rot="R90"/>
-<instance part="ANT1" gate="2450AT45A100" x="210.82" y="149.86"/>
+<instance part="ANT1" gate="2450AT45A100" x="233.68" y="142.24"/>
 <instance part="GND10" gate="1" x="157.48" y="205.74" rot="MR0"/>
 <instance part="F1" gate="2450FM07A0029" x="137.16" y="220.98"/>
@@
 <instance part="SWDIO" gate="G$1" x="259.08" y="200.66" rot="R90"/>
 <instance part="GND" gate="G$1" x="259.08" y="167.64" rot="R90"/>
-<instance part="VDD" gate="G$1" x="259.08" y="160.02" rot="R90"/>
 <instance part="SWO" gate="G$1" x="259.08" y="208.28" rot="R90"/>
-<instance part="VDD_11" gate="1" x="274.32" y="162.56"/>
+<instance part="GND12" gate="1" x="213.36" y="116.84"/>
+<instance part="R16" gate="G$1" x="210.82" y="139.7"/>
+<instance part="R17" gate="G$1" x="220.98" y="129.54" rot="R90"/>
+<instance part="R18" gate="G$1" x="203.2" y="129.54" rot="R90"/>
 </instances>
 <busses>
@@
 <label x="261.62" y="167.64" size="1.778" layer="95" xref="yes"/>
 </segment>
+<segment>
+<pinref part="R18" gate="G$1" pin="1"/>
+<wire x1="203.2" y1="124.46" x2="203.2" y2="121.92" width="0.1524" layer="91"/>
+<wire x1="203.2" y1="121.92" x2="213.36" y2="121.92" width="0.1524" layer="91"/>
+<pinref part="R17" gate="G$1" pin="1"/>
+<wire x1="213.36" y1="121.92" x2="220.98" y2="121.92" width="0.1524" layer="91"/>
+<wire x1="220.98" y1="121.92" x2="220.98" y2="124.46" width="0.1524" layer="91"/>
+<pinref part="GND12" gate="1" pin="GND"/>
+<wire x1="213.36" y1="119.38" x2="213.36" y2="121.92" width="0.1524" layer="91"/>
+<junction x="213.36" y="121.92"/>
+</segment>
 </net>
 <net name="DEC1" class="0">
@@
 </segment>
 <segment>
-<pinref part="ANT1" gate="2450AT45A100" pin="1"/>
-<wire x1="200.66" y1="147.32" x2="193.04" y2="147.32" width="0.1524" layer="91"/>
-<label x="193.04" y="147.32" size="1.27" layer="95" rot="R180" xref="yes"/>
+<pinref part="R16" gate="G$1" pin="1"/>
+<wire x1="205.74" y1="139.7" x2="203.2" y2="139.7" width="0.1524" layer="91"/>
+<pinref part="R18" gate="G$1" pin="2"/>
+<wire x1="203.2" y1="139.7" x2="193.04" y2="139.7" width="0.1524" layer="91"/>
+<wire x1="203.2" y1="134.62" x2="203.2" y2="139.7" width="0.1524" layer="91"/>
+<junction x="203.2" y="139.7"/>
+<label x="193.04" y="139.7" size="1.778" layer="95" rot="R180" xref="yes"/>
 </segment>
 </net>
@@
 <wire x1="-81.28" y1="124.46" x2="-81.28" y2="129.54" width="0.1524" layer="91"/>
 </segment>
-<segment>
-<pinref part="VDD" gate="G$1" pin="P$1"/>
-<pinref part="VDD_11" gate="1" pin="V+"/>
-<wire x1="259.08" y1="160.02" x2="274.32" y2="160.02" width="0.1524" layer="91"/>
-</segment>
 </net>
 <net name="N$1" class="0">
@@
 </segment>
 </net>
+<net name="N$18" class="0">
+<segment>
+<pinref part="ANT1" gate="2450AT45A100" pin="1"/>
+<pinref part="R16" gate="G$1" pin="2"/>
+<wire x1="223.52" y1="139.7" x2="220.98" y2="139.7" width="0.1524" layer="91"/>
+<pinref part="R17" gate="G$1" pin="2"/>
+<wire x1="220.98" y1="139.7" x2="215.9" y2="139.7" width="0.1524" layer="91"/>
+<wire x1="220.98" y1="134.62" x2="220.98" y2="139.7" width="0.1524" layer="91"/>
+<junction x="220.98" y="139.7"/>
+</segment>
+</net>

Commit message: UPD: battery
Parts:
- removed H1: HDC1080, tilesPartComp:HDC1080
- added HU1: HDC2010, tilesPartComp:HDC2010
- R4: value 10K -> 37K
- U$14: value GM351824 -> GM171538; device tilesPartComp:GM351824 -> tilesPartComp:GM171538
Connections:
- net N$16 renamed CBAT
- net GND: now also HU1.GND; no longer H1.GND
- net P0.25: now also HU1.SDA; no longer H1.SDA
- net P0.26: now also HU1.SCL; no longer H1.SCL
- net V+: now also HU1.ADDR, HU1.VDD; no longer H1.VDD
Other:
- note added: "37K = 27mA"
- note added: "I2C = 0x40"
- note added: "I2C = 0x41"
Changed lines of the file:
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@@
 <part name="R3" library="rcl" library_urn="urn:adsk.eagle:library:334" deviceset="R-EU_" device="R0603" package3d_urn="urn:adsk.eagle:package:23555/2" value="200"/>
 <part name="C3" library="rcl" library_urn="urn:adsk.eagle:library:334" deviceset="C-EU" device="C0805" package3d_urn="urn:adsk.eagle:package:23617/2" value="10µF"/>
-<part name="R4" library="rcl" library_urn="urn:adsk.eagle:library:334" deviceset="R-EU_" device="R0603" package3d_urn="urn:adsk.eagle:package:23555/2" value="10K"/>
+<part name="R4" library="rcl" library_urn="urn:adsk.eagle:library:334" deviceset="R-EU_" device="R0603" package3d_urn="urn:adsk.eagle:package:23555/2" value="37K"/>
 <part name="U7" library="tilesPartComp" deviceset="CP2102N-A01-GQFN24" device=""/>
 <part name="U$8" library="tilesPartComp" deviceset="VUSB" device=""/>
@@
 <part name="DSG" library="tilesPartComp" deviceset="CSD16406Q3" device=""/>
 <part name="U12" library="tilesPartComp" deviceset="BQ297XY" device=""/>
-<part name="U$14" library="tilesPartComp" deviceset="GM351824" device=""/>
+<part name="U$14" library="tilesPartComp" deviceset="GM171538" device=""/>
 <part name="ANT1" library="tilesPartComp" deviceset="2450AT45A100" device=""/>
 <part name="GND10" library="supply1" deviceset="GND" device=""/>
@@
 <part name="VDD_9" library="supply2" library_urn="urn:adsk.eagle:library:372" deviceset="V+" device="" value="3.3V"/>
 <part name="GND14" library="supply1" deviceset="GND" device=""/>
-<part name="H1" library="tilesPartComp" deviceset="HDC1080" device=""/>
 <part name="GND15" library="supply1" deviceset="GND" device=""/>
 <part name="GND16" library="supply1" deviceset="GND" device=""/>
@@
 <part name="R17" library="rcl" library_urn="urn:adsk.eagle:library:334" deviceset="R-EU_" device="R0402" package3d_urn="urn:adsk.eagle:package:23547/2" value="DNP"/>
 <part name="R18" library="rcl" library_urn="urn:adsk.eagle:library:334" deviceset="R-EU_" device="R0402" package3d_urn="urn:adsk.eagle:package:23547/2" value="DNP"/>
+<part name="HU1" library="tilesPartComp" deviceset="HDC2010" device=""/>
 </parts>
 <sheets>
@@
 <text x="121.92" y="360.68" size="1.778" layer="97">1.0K  = 1000mA</text>
 <text x="121.92" y="370.84" size="1.778" layer="97">20K  = 50mA</text>
-<text x="127" y="375.92" size="1.27" layer="97">R-PROG</text>
+<text x="127" y="378.46" size="1.27" layer="97">R-PROG</text>
 <text x="-121.92" y="274.32" size="2.54" layer="91">Battery protection</text>
 <text x="-101.6" y="248.92" size="1.27" layer="91">TI bq2970, bq2971, bq2972, bq2973
@@
 ADC value at 2.7 V - 12 bit setup: 1.93 V * (1/5) / 0.6 V * 4095 = 2634
 Usable ADC resolution - 12 bit setup: 4095 - 2634 = 1461</text>
+<text x="15.24" y="147.32" size="1.778" layer="91">I2C = 0x40</text>
+<text x="12.7" y="116.84" size="1.778" layer="91">I2C = 0x41</text>
+<text x="121.92" y="373.38" size="1.778" layer="97">37K  = 27mA</text>
 </plain>
 <instances>
@@
 <instance part="DSG" gate="CSD16406Q3" x="-134.62" y="210.82" rot="MR270"/>
 <instance part="U12" gate="BQ297XY" x="-96.52" y="233.68"/>
-<instance part="U$14" gate="G$1" x="-40.64" y="233.68" rot="R90"/>
+<instance part="U$14" gate="GM171538" x="-40.64" y="233.68" rot="R90"/>
 <instance part="ANT1" gate="2450AT45A100" x="233.68" y="142.24"/>
 <instance part="GND10" gate="1" x="157.48" y="205.74" rot="MR0"/>
@@
 <instance part="VDD_9" gate="1" x="48.26" y="162.56"/>
 <instance part="GND14" gate="1" x="-7.62" y="127" rot="MR0"/>
-<instance part="H1" gate="HDC1080" x="10.16" y="104.14"/>
 <instance part="GND15" gate="1" x="-7.62" y="91.44" rot="MR0"/>
 <instance part="GND16" gate="1" x="40.64" y="119.38" rot="MR0"/>
@@
 <instance part="R17" gate="G$1" x="220.98" y="129.54" rot="R90"/>
 <instance part="R18" gate="G$1" x="203.2" y="129.54" rot="R90"/>
+<instance part="HU1" gate="HDC2010" x="10.16" y="106.68"/>
 </instances>
 <busses>
@@
 </segment>
 <segment>
-<pinref part="H1" gate="HDC1080" pin="GND"/>
-<wire x1="-5.08" y1="104.14" x2="-7.62" y2="104.14" width="0.1524" layer="91"/>
+<wire x1="-5.08" y1="106.68" x2="-7.62" y2="106.68" width="0.1524" layer="91"/>
 <pinref part="GND15" gate="1" pin="GND"/>
-<wire x1="-7.62" y1="104.14" x2="-7.62" y2="93.98" width="0.1524" layer="91"/>
+<wire x1="-7.62" y1="106.68" x2="-7.62" y2="93.98" width="0.1524" layer="91"/>
+<pinref part="HU1" gate="HDC2010" pin="GND"/>
 </segment>
 <segment>
@@
 </segment>
 <segment>
-<pinref part="H1" gate="HDC1080" pin="SCL"/>
-<wire x1="25.4" y1="109.22" x2="30.48" y2="109.22" width="0.1524" layer="91"/>
 <pinref part="T1" gate="SI7051-A20" pin="SCL"/>
 <wire x1="30.48" y1="142.24" x2="25.4" y2="142.24" width="0.1524" layer="91"/>
 <wire x1="30.48" y1="142.24" x2="30.48" y2="139.7" width="0.1524" layer="91"/>
-<wire x1="30.48" y1="139.7" x2="30.48" y2="109.22" width="0.1524" layer="91"/>
+<wire x1="30.48" y1="139.7" x2="30.48" y2="111.76" width="0.1524" layer="91"/>
 <wire x1="30.48" y1="139.7" x2="35.56" y2="139.7" width="0.1524" layer="91"/>
 <junction x="30.48" y="139.7"/>
@@
 <label x="38.1" y="139.7" size="1.27" layer="95" xref="yes"/>
 <pinref part="R9" gate="G$1" pin="1"/>
+<pinref part="HU1" gate="HDC2010" pin="SCL"/>
+<wire x1="25.4" y1="111.76" x2="30.48" y2="111.76" width="0.1524" layer="91"/>
 </segment>
 </net>
@@
 <segment>
 <label x="-22.86" y="139.7" size="1.27" layer="95" rot="R180" xref="yes"/>
-<pinref part="H1" gate="HDC1080" pin="SDA"/>
 <wire x1="-12.7" y1="139.7" x2="-17.78" y2="139.7" width="0.1524" layer="91"/>
 <wire x1="-17.78" y1="139.7" x2="-22.86" y2="139.7" width="0.1524" layer="91"/>
-<wire x1="-12.7" y1="139.7" x2="-12.7" y2="109.22" width="0.1524" layer="91"/>
-<wire x1="-12.7" y1="109.22" x2="-5.08" y2="109.22" width="0.1524" layer="91"/>
+<wire x1="-12.7" y1="139.7" x2="-12.7" y2="111.76" width="0.1524" layer="91"/>
+<wire x1="-12.7" y1="111.76" x2="-5.08" y2="111.76" width="0.1524" layer="91"/>
 <wire x1="-17.78" y1="144.78" x2="-17.78" y2="139.7" width="0.1524" layer="91"/>
 <junction x="-17.78" y="139.7"/>
@@
 <junction x="-12.7" y="139.7"/>
 <pinref part="R15" gate="G$1" pin="1"/>
+<pinref part="HU1" gate="HDC2010" pin="SDA"/>
 </segment>
 </net>
@@
 <pinref part="T1" gate="SI7051-A20" pin="VDD"/>
 <wire x1="25.4" y1="137.16" x2="40.64" y2="137.16" width="0.1524" layer="91"/>
-<pinref part="H1" gate="HDC1080" pin="VDD"/>
 <wire x1="40.64" y1="137.16" x2="48.26" y2="137.16" width="0.1524" layer="91"/>
 <wire x1="25.4" y1="104.14" x2="40.64" y2="104.14" width="0.1524" layer="91"/>
@@
 <wire x1="40.64" y1="101.6" x2="40.64" y2="104.14" width="0.1524" layer="91"/>
 <junction x="40.64" y="104.14"/>
+<pinref part="HU1" gate="HDC2010" pin="ADDR"/>
+<wire x1="25.4" y1="104.14" x2="25.4" y2="106.68" width="0.1524" layer="91"/>
+<pinref part="HU1" gate="HDC2010" pin="VDD"/>
+<wire x1="25.4" y1="104.14" x2="25.4" y2="101.6" width="0.1524" layer="91"/>
+<junction x="25.4" y="104.14"/>
 </segment>
 <segment>
@@
 </segment>
 </net>
-<net name="N$16" class="0">
+<net name="CBAT" class="0">
 <segment>
 <pinref part="C7" gate="G$1" pin="2"/>
 <wire x1="-58.42" y1="208.28" x2="-58.42" y2="218.44" width="0.1524" layer="91"/>
-<pinref part="U$14" gate="G$1" pin="-"/>
+<pinref part="U$14" gate="GM171538" pin="-"/>
 <wire x1="-40.64" y1="231.14" x2="-40.64" y2="208.28" width="0.1524" layer="91"/>
 <wire x1="-40.64" y1="208.28" x2="-58.42" y2="208.28" width="0.1524" layer="91"/>
@@
 <wire x1="-40.64" y1="264.16" x2="-58.42" y2="264.16" width="0.1524" layer="91"/>
 <junction x="-58.42" y="264.16"/>
-<pinref part="U$14" gate="G$1" pin="+"/>
-</segment>
-<segment>
+<pinref part="U$14" gate="GM171538" pin="+"/>
+</segment>
+<segment>

Commit message: UPD: finished before moving left area
Parts:
- removed C7: 0.1µF, rcl:C-EUC0603K
- removed CHG, DSG: CSD16406Q3, tilesPartComp:CSD16406Q3
- removed R7: 330, rcl:R-EU_R0603
- removed R8: 2.2K, rcl:R-EU_R0603
- removed U$14: GM171538, tilesPartComp:GM171538
- removed U12: BQ297XY, tilesPartComp:BQ297XY
- added TEST1, TEST2: TESTPOINT_SQUARE_SMT, tilesPartComp:TESTPOINT_SQUARE_SMT
Connections:
- removed net CBAT: C7.2, DSG.S, U$14.-, U12.VSS
- removed net N$11: CHG.D, DSG.D
- removed net N$12: DSG.G, U12.DOUT
- removed net N$13: C7.1, R7.2, U12.BAT
- removed net N$14: CHG.G, U12.COUT
- removed net N$15: R8.1, U12.V-
- net GND: now also TEST2.P; no longer CHG.S, R8.2
- net VBAT: now also TEST1.P; no longer R7.1, U$14.+
Other:
- note added: "Battery"
- note removed: "Battery protection"
- note removed: "TI bq2970, bq2971, bq2972, bq2973 depending on battery parameters"
Changed lines of the file:
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@@
 <part name="GND13" library="supply1" library_urn="urn:adsk.eagle:library:371" deviceset="GND" device=""/>
 <part name="U$10" library="tilesPartComp" deviceset="VBAT" device=""/>
-<part name="C7" library="rcl" library_urn="urn:adsk.eagle:library:334" deviceset="C-EU" device="C0603K" package3d_urn="urn:adsk.eagle:package:23680/2" value="0.1µF"/>
-<part name="R7" library="rcl" library_urn="urn:adsk.eagle:library:334" deviceset="R-EU_" device="R0603" package3d_urn="urn:adsk.eagle:package:23555/2" value="330"/>
-<part name="R8" library="rcl" library_urn="urn:adsk.eagle:library:334" deviceset="R-EU_" device="R0603" package3d_urn="urn:adsk.eagle:package:23555/2" value="2.2K"/>
-<part name="CHG" library="tilesPartComp" deviceset="CSD16406Q3" device=""/>
-<part name="DSG" library="tilesPartComp" deviceset="CSD16406Q3" device=""/>
-<part name="U12" library="tilesPartComp" deviceset="BQ297XY" device=""/>
-<part name="U$14" library="tilesPartComp" deviceset="GM171538" device=""/>
 <part name="ANT1" library="tilesPartComp" deviceset="2450AT45A100" device=""/>
 <part name="GND10" library="supply1" deviceset="GND" device=""/>
@@
 <part name="R18" library="rcl" library_urn="urn:adsk.eagle:library:334" deviceset="R-EU_" device="R0402" package3d_urn="urn:adsk.eagle:package:23547/2" value="DNP"/>
 <part name="HU1" library="tilesPartComp" deviceset="HDC2010" device=""/>
+<part name="TEST1" library="tilesPartComp" deviceset="TESTPOINT_SQUARE_SMT" device=""/>
+<part name="TEST2" library="tilesPartComp" deviceset="TESTPOINT_SQUARE_SMT" device=""/>
 </parts>
 <sheets>
@@
 <text x="121.92" y="370.84" size="1.778" layer="97">20K  = 50mA</text>
 <text x="127" y="378.46" size="1.27" layer="97">R-PROG</text>
-<text x="-121.92" y="274.32" size="2.54" layer="91">Battery protection</text>
-<text x="-101.6" y="248.92" size="1.27" layer="91">TI bq2970, bq2971, bq2972, bq2973
-depending on battery parameters</text>
+<text x="-66.04" y="261.62" size="2.54" layer="91">Battery</text>
 <text x="88.9" y="363.22" size="1.27" layer="91">Check charge V based on battery type</text>
 <text x="2.54" y="162.56" size="1.778" layer="94">Temperature and Humidity sensors</text>
@@
 <instance part="FRST" gate="G$1" x="259.08" y="182.88" rot="R90"/>
 <instance part="DFU" gate="G$1" x="259.08" y="175.26" rot="R90"/>
-<instance part="GND13" gate="1" x="-177.8" y="198.12"/>
-<instance part="U$10" gate="G$1" x="-58.42" y="274.32"/>
-<instance part="C7" gate="G$1" x="-58.42" y="223.52"/>
-<instance part="R7" gate="G$1" x="-58.42" y="248.92" rot="R270"/>
-<instance part="R8" gate="G$1" x="-177.8" y="233.68" rot="R270"/>
-<instance part="CHG" gate="CSD16406Q3" x="-157.48" y="210.82" rot="R270"/>
-<instance part="DSG" gate="CSD16406Q3" x="-134.62" y="210.82" rot="MR270"/>
-<instance part="U12" gate="BQ297XY" x="-96.52" y="233.68"/>
-<instance part="U$14" gate="GM171538" x="-40.64" y="233.68" rot="R90"/>
+<instance part="GND13" gate="1" x="-60.96" y="233.68"/>
+<instance part="U$10" gate="G$1" x="-45.72" y="243.84"/>
 <instance part="ANT1" gate="2450AT45A100" x="233.68" y="142.24"/>
 <instance part="GND10" gate="1" x="157.48" y="205.74" rot="MR0"/>
@@
 <instance part="R18" gate="G$1" x="203.2" y="129.54" rot="R90"/>
 <instance part="HU1" gate="HDC2010" x="10.16" y="106.68"/>
+<instance part="TEST1" gate="G$1" x="-53.34" y="254"/>
+<instance part="TEST2" gate="G$1" x="-60.96" y="254"/>
 </instances>
 <busses>
@@
 <pinref part="GND11" gate="1" pin="GND"/>
 <wire x1="226.06" y1="210.82" x2="226.06" y2="208.28" width="0.1524" layer="91"/>
-</segment>
-<segment>
-<pinref part="GND13" gate="1" pin="GND"/>
-<pinref part="R8" gate="G$1" pin="2"/>
-<wire x1="-177.8" y1="228.6" x2="-177.8" y2="208.28" width="0.1524" layer="91"/>
-<pinref part="CHG" gate="CSD16406Q3" pin="S"/>
-<wire x1="-177.8" y1="208.28" x2="-177.8" y2="200.66" width="0.1524" layer="91"/>
-<wire x1="-167.64" y1="208.28" x2="-177.8" y2="208.28" width="0.1524" layer="91"/>
-<junction x="-177.8" y="208.28"/>
 </segment>
 <segment>
@@
 <wire x1="213.36" y1="119.38" x2="213.36" y2="121.92" width="0.1524" layer="91"/>
 <junction x="213.36" y="121.92"/>
+</segment>
+<segment>
+<pinref part="GND13" gate="1" pin="GND"/>
+<pinref part="TEST2" gate="G$1" pin="P"/>
+<wire x1="-60.96" y1="246.38" x2="-60.96" y2="236.22" width="0.1524" layer="91"/>
 </segment>
 </net>
@@
 </segment>
 </net>
-<net name="N$13" class="0">
-<segment>
-<pinref part="U12" gate="BQ297XY" pin="BAT"/>
-<wire x1="-71.12" y1="233.68" x2="-58.42" y2="233.68" width="0.1524" layer="91"/>
-<pinref part="R7" gate="G$1" pin="2"/>
-<wire x1="-58.42" y1="233.68" x2="-58.42" y2="243.84" width="0.1524" layer="91"/>
-<pinref part="C7" gate="G$1" pin="1"/>
-<wire x1="-58.42" y1="233.68" x2="-58.42" y2="226.06" width="0.1524" layer="91"/>
-<junction x="-58.42" y="233.68"/>
-</segment>
-</net>
-<net name="N$15" class="0">
-<segment>
-<pinref part="U12" gate="BQ297XY" pin="V-"/>
-<wire x1="-71.12" y1="241.3" x2="-66.04" y2="241.3" width="0.1524" layer="91"/>
-<wire x1="-66.04" y1="241.3" x2="-66.04" y2="256.54" width="0.1524" layer="91"/>
-<wire x1="-66.04" y1="256.54" x2="-177.8" y2="256.54" width="0.1524" layer="91"/>
-<wire x1="-177.8" y1="256.54" x2="-177.8" y2="238.76" width="0.1524" layer="91"/>
-<pinref part="R8" gate="G$1" pin="1"/>
-</segment>
-</net>
-<net name="CBAT" class="0">
-<segment>
-<pinref part="C7" gate="G$1" pin="2"/>
-<wire x1="-58.42" y1="208.28" x2="-58.42" y2="218.44" width="0.1524" layer="91"/>
-<pinref part="U$14" gate="GM171538" pin="-"/>
-<wire x1="-40.64" y1="231.14" x2="-40.64" y2="208.28" width="0.1524" layer="91"/>
-<wire x1="-40.64" y1="208.28" x2="-58.42" y2="208.28" width="0.1524" layer="91"/>
-<wire x1="-58.42" y1="208.28" x2="-66.04" y2="208.28" width="0.1524" layer="91"/>
-<junction x="-58.42" y="208.28"/>
-<pinref part="U12" gate="BQ297XY" pin="VSS"/>
-<wire x1="-71.12" y1="226.06" x2="-66.04" y2="226.06" width="0.1524" layer="91"/>
-<wire x1="-66.04" y1="226.06" x2="-66.04" y2="208.28" width="0.1524" layer="91"/>
-<pinref part="DSG" gate="CSD16406Q3" pin="S"/>
-<wire x1="-124.46" y1="208.28" x2="-66.04" y2="208.28" width="0.1524" layer="91"/>
-<junction x="-66.04" y="208.28"/>
-</segment>
-</net>
-<net name="N$11" class="0">
-<segment>
-<pinref part="CHG" gate="CSD16406Q3" pin="D"/>
-<pinref part="DSG" gate="CSD16406Q3" pin="D"/>
-<wire x1="-149.86" y1="208.28" x2="-142.24" y2="208.28" width="0.1524" layer="91"/>
-</segment>
-</net>
-<net name="N$12" class="0">
-<segment>
-<pinref part="DSG" gate="CSD16406Q3" pin="G"/>
-<wire x1="-132.08" y1="218.44" x2="-132.08" y2="226.06" width="0.1524" layer="91"/>
-<pinref part="U12" gate="BQ297XY" pin="DOUT"/>
-<wire x1="-132.08" y1="226.06" x2="-121.92" y2="226.06" width="0.1524" layer="91"/>
-</segment>
-</net>
-<net name="N$14" class="0">
-<segment>
-<pinref part="U12" gate="BQ297XY" pin="COUT"/>
-<wire x1="-121.92" y1="233.68" x2="-160.02" y2="233.68" width="0.1524" layer="91"/>
-<pinref part="CHG" gate="CSD16406Q3" pin="G"/>
-<wire x1="-160.02" y1="233.68" x2="-160.02" y2="218.44" width="0.1524" layer="91"/>
-</segment>
-</net>
 <net name="N$17" class="0">
 <segment>
@@
 </net>
 <net name="VBAT" class="0">
-<segment>
-<pinref part="U$10" gate="G$1" pin="VBAT"/>
-<wire x1="-58.42" y1="271.78" x2="-58.42" y2="264.16" width="0.1524" layer="91"/>
-<wire x1="-58.42" y1="264.16" x2="-58.42" y2="254" width="0.1524" layer="91"/>
-<pinref part="R7" gate="G$1" pin="1"/>
-<wire x1="-40.64" y1="236.22" x2="-40.64" y2="264.16" width="0.1524" layer="91"/>
-<wire x1="-40.64" y1="264.16" x2="-58.42" y2="264.16" width="0.1524" layer="91"/>
-<junction x="-58.42" y="264.16"/>
-<pinref part="U$14" gate="GM171538" pin="+"/>
-</segment>
 <segment>
 <pinref part="U$9" gate="G$1" pin="VBAT"/>
@@
 <junction x="147.32" y="353.06"/>
 </segment>
-</net>
+<segment>
+<pinref part="U$10" gate="G$1" pin="VBAT"/>
+<wire x1="-53.34" y1="236.22" x2="-45.72" y2="236.22" width="0.1524" layer="91"/>
+<wire x1="-45.72" y1="236.22" x2="-45.72" y2="241.3" width="0.1524" layer="91"/>
+<pinref part="TEST1" gate="G$1" pin="P"/>
+<wire x1="-53.34" y1="246.38" x2="-53.34" y2="236.22" width="0.1524" layer="91"/>
+</segment>
+</net>
